File: nutrino.brd (EAGLE design)
At the start: 160 x 100 mm, 94 parts, among them CN1 STEREO-3.5-MJ8435, CON1 MINI-USB-, IC1 TLV61046A, IC2 TAR5SB33, IC3 PCM2704, IC4 NJM4580EMP8, Q1 12M, SW1 TOGGLESW_SLIMPANEL, SW2 TOGGLESW_SLIMPANEL

Commit message: placed parts
Parts:
- removed 100K, 100K1: 10k, Passive_Robotech:2012-R
- added HOLE1, HOLE2, HOLE3, HOLE4: HOLE_3.2, Document_Robotech:HOLE_3.2
- added R33, R34: 100k, Passive_Robotech:2012-R
- SW1, SW2: value TOGGLESW_SLIMPANEL -> SLIDESW_SS12D01G4; device Passive_Robotech:TOGGLESW_PANEL -> Passive_Robotech:SS12D01G4
- U1: device rezzonics:NUTUBE_6P1 -> rezzonics:NUTUBE_6P1_1
- moved R13 152.3 mm to (37.8, 6.35), turned to 90 degrees
- moved C39 151.3 mm to (54.1, 34.3), turned to 90 degrees
- moved R32 148.4 mm to (57.9, 8.89), turned to 180 degrees
- moved CN1 147.9 mm to (60.1, 14.5), turned to 270 degrees
- moved C34 142.5 mm to (53.6, 45.5), turned to 90 degrees
- moved VR5 139.6 mm to (58.1, 32.0), turned to 90 degrees
- moved R15 138.8 mm to (21.1, 17.0), turned to 180 degrees
- moved U$3 138.6 mm to (37.1, 21.8), turned to 90 degrees
- moved C35 133.8 mm to (43.9, 40.1), turned to 90 degrees
- moved C17 133.1 mm to (17.5, 17.0), turned to 180 degrees
- moved C13 131.8 mm to (18.3, 4.32), turned to 180 degrees
- moved R12 131.3 mm to (37.3, 42.2), turned to 270 degrees
- moved C24 131.0 mm to (35.1, 6.35), turned to 90 degrees
- moved C33 130.5 mm to (46.2, 25.1), turned to 90 degrees
- moved R30 129.9 mm to (54.1, 30.7), turned to 270 degrees
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Connections:
- removed net POWER-GND: C10.2, C8.2, C9.2, IC2.2
- net FET_L: now also SW1.P$2; no longer SW1.2
- net FET_R: now also SW2.P$2; no longer SW2.2
- net GND: now also C10.2, C8.2, C9.2, IC2.2
- net N$24: now also SW1.P$1; no longer SW1.1
- net N$25: now also SW1.P$3; no longer SW1.3
- net N$29: now also SW2.P$1; no longer SW2.1
- net N$30: now also SW2.P$3; no longer SW2.3
- net N$34: now also R34.1; no longer 100K.1
- net N$35: now also R34.2; no longer 100K.2
- net N$42: now also R33.1; no longer 100K1.1
- net N$43: now also R33.2; no longer 100K1.2
Other:
- board size 160 x 100 mm -> 65 x 50 mm

Commit message: Board diagram completed
Parts:
- moved C7 52.6 mm to (41.7, 19.3), flipped to the bottom, turned to 90 degrees
- moved C6 42.8 mm to (48.0, 34.3), flipped to the bottom, turned to 270 degrees
- moved C5 42.5 mm to (35.8, 23.6), flipped to the bottom, turned to 270 degrees
- moved C4 33.4 mm to (35.8, 32.0), flipped to the bottom, turned to 90 degrees
- moved C14 31.5 mm to (5.59, 17.8), turned to 180 degrees
- moved C9 5.89 mm to (6.10, 41.9), turned to 0 degrees
- moved R2 5.89 mm to (12.2, 37.3), turned to 180 degrees
- moved R11 5.85 mm to (19.8, 18.3)
- moved C19 5.34 mm to (19.8, 23.9), flipped to the top, turned to 180 degrees
- moved R8 5.34 mm to (16.0, 23.9), flipped to the top, turned to 180 degrees
- moved R15 5.14 mm to (20.3, 11.9), turned to 270 degrees
- moved R1 4.33 mm to (12.2, 32.0), turned to 0 degrees
- moved C3 3.97 mm to (12.2, 34.8), turned to 180 degrees
- moved C1 3.59 mm to (16.0, 28.2), turned to 0 degrees
- moved C2 3.31 mm to (12.2, 29.2), turned to 180 degrees
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Connections:
- removed net +26V: C4.1, C5.1, C6.1, C7.1
- net AVCC: now also C4.1, C5.1, C6.1, C7.1
- net GND: now also CON1.M1, CON1.M2, CON1.M3, CON1.M4
- net N$20: now also VR1.2, VR1.BR; no longer VR1.1
- net N$26: now also VR2.1, VR2.BR; no longer VR2.2
- net TUBE_L: now also VR1.1; no longer VR1.2
- net TUBE_R: now also VR2.2; no longer VR2.1
Routing:
- net AVCC: track 0.00 -> 140.9 mm, vias 0 -> 8
- net +3V3: track 0.00 -> 121.8 mm, vias 0 -> 2
- net +5V: track 0.00 -> 74.4 mm, vias 0 -> 2
- net N$36: track 0.00 -> 59.7 mm
- net N$44: track 0.00 -> 39.0 mm, vias 0 -> 3
- net FET_R: track 0.00 -> 36.9 mm
- net N$10: track 0.00 -> 35.3 mm
- net N$18: track 0.00 -> 34.1 mm
- net N$42: track 0.00 -> 31.6 mm
- net FET_L: track 0.00 -> 30.9 mm
- net BIAS: track 0.00 -> 28.0 mm, vias 0 -> 1
- net DAC_R: track 0.00 -> 23.1 mm
- net N$5: track 0.00 -> 21.1 mm, vias 0 -> 2
- net N$6: track 0.00 -> 20.7 mm, vias 0 -> 2
- net N$40: track 0.00 -> 19.9 mm
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- added copper zone on layer 1, net GND
- added copper zone on layer 16, net GND
Other:
- board text added: "2023 Hamataku lab."
- board text added: "Nutrino"
- board text added: "ver1.0"

Commit message: add image
Parts:
- VR5: value (none) -> 100K
Changed lines of the file:
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@@
 <grid distance="10" unitdist="mil" unit="mil" style="lines" multiple="1" display="yes" altdistance="5" altunitdist="mil" altunit="mil"/>
 <layers>
-<layer number="1" name="Top" color="4" fill="1" visible="no" active="yes"/>
+<layer number="1" name="Top" color="4" fill="1" visible="yes" active="yes"/>
 <layer number="2" name="Route2" color="16" fill="1" visible="no" active="no"/>
 <layer number="3" name="Route3" color="17" fill="1" visible="no" active="no"/>
@@
 <layer number="14" name="Route14" color="22" fill="1" visible="no" active="no"/>
 <layer number="15" name="Route15" color="23" fill="1" visible="no" active="no"/>
-<layer number="16" name="Bottom" color="1" fill="1" visible="yes" active="yes"/>
+<layer number="16" name="Bottom" color="1" fill="1" visible="no" active="yes"/>
 <layer number="17" name="Pads" color="2" fill="1" visible="yes" active="yes"/>
 <layer number="18" name="Vias" color="2" fill="1" visible="yes" active="yes"/>
 <layer number="19" name="Unrouted" color="6" fill="1" visible="yes" active="yes"/>
 <layer number="20" name="Dimension" color="24" fill="1" visible="yes" active="yes"/>
-<layer number="21" name="tPlace" color="7" fill="1" visible="no" active="yes"/>
-<layer number="22" name="bPlace" color="7" fill="1" visible="yes" active="yes"/>
-<layer number="23" name="tOrigins" color="15" fill="1" visible="no" active="yes"/>
-<layer number="24" name="bOrigins" color="15" fill="1" visible="yes" active="yes"/>
+<layer number="21" name="tPlace" color="7" fill="1" visible="yes" active="yes"/>
+<layer number="22" name="bPlace" color="7" fill="1" visible="no" active="yes"/>
+<layer number="23" name="tOrigins" color="15" fill="1" visible="yes" active="yes"/>
+<layer number="24" name="bOrigins" color="15" fill="1" visible="no" active="yes"/>
 <layer number="25" name="tNames" color="7" fill="1" visible="no" active="yes"/>
 <layer number="26" name="bNames" color="7" fill="1" visible="no" active="yes"/>
-<layer number="27" name="tValues" color="7" fill="1" visible="no" active="yes"/>
-<layer number="28" name="bValues" color="7" fill="1" visible="yes" active="yes"/>
+<layer number="27" name="tValues" color="7" fill="1" visible="yes" active="yes"/>
+<layer number="28" name="bValues" color="7" fill="1" visible="no" active="yes"/>
 <layer number="29" name="tStop" color="7" fill="3" visible="no" active="yes"/>
 <layer number="30" name="bStop" color="7" fill="6" visible="no" active="yes"/>
@@
 <layer number="37" name="tTest" color="7" fill="1" visible="no" active="yes"/>
 <layer number="38" name="bTest" color="7" fill="1" visible="no" active="yes"/>
-<layer number="39" name="tKeepout" color="4" fill="11" visible="no" active="yes"/>
-<layer number="40" name="bKeepout" color="1" fill="11" visible="yes" active="yes"/>
-<layer number="41" name="tRestrict" color="4" fill="10" visible="no" active="yes"/>
-<layer number="42" name="bRestrict" color="1" fill="10" visible="yes" active="yes"/>
+<layer number="39" name="tKeepout" color="4" fill="11" visible="yes" active="yes"/>
+<layer number="40" name="bKeepout" color="1" fill="11" visible="no" active="yes"/>
+<layer number="41" name="tRestrict" color="4" fill="10" visible="yes" active="yes"/>
+<layer number="42" name="bRestrict" color="1" fill="10" visible="no" active="yes"/>
 <layer number="43" name="vRestrict" color="2" fill="10" visible="no" active="yes"/>
 <layer number="44" name="Drills" color="7" fill="1" visible="no" active="yes"/>
@@
 <layer number="49" name="Reference" color="7" fill="1" visible="no" active="yes"/>
 <layer number="50" name="dxf" color="7" fill="1" visible="no" active="no"/>
-<layer number="51" name="tDocu" color="7" fill="1" visible="no" active="yes"/>
-<layer number="52" name="bDocu" color="7" fill="1" visible="yes" active="yes"/>
+<layer number="51" name="tDocu" color="7" fill="1" visible="yes" active="yes"/>
+<layer number="52" name="bDocu" color="7" fill="1" visible="no" active="yes"/>
 <layer number="53" name="tGND_GNDA" color="7" fill="1" visible="no" active="no"/>
 <layer number="54" name="bGND_GNDA" color="7" fill="1" visible="no" active="no"/>
@@
 <attribute name="VALUE" x="28.956" y="1.524" size="1.27" layer="27" font="vector" rot="R90"/>
 </element>
-<element name="VR5" library="Passive_Robotech" package="VR2C" value="" x="58.086" y="32.004" smashed="yes" rot="R90">
+<element name="VR5" library="Passive_Robotech" package="VR2C" value="100K" x="58.086" y="32.004" smashed="yes" rot="R90">
 <attribute name="NAME" x="56.816" y="30.734" size="1.27" layer="25" rot="R90"/>
-<attribute name="VALUE" x="63.166" y="30.734" size="1.27" layer="27" rot="R90"/>
+<attribute name="VALUE" x="63.674" y="32.512" size="1.27" layer="27" rot="R90"/>
 </element>
 <element name="IC3" library="IC_Robotech" package="SSOP28" value="PCM2704" x="13.716" y="8.89" smashed="yes">
@@
 <wire x1="58.086" y1="34.544" x2="58.086" y2="37.084" width="0.3048" layer="1"/>
 <wire x1="51.8476" y1="29.464" x2="52.8636" y2="30.48" width="0.3048" layer="1"/>
-<wire x1="58.086" y1="33.85153125" x2="58.086" y2="34.544" width="0.3048" layer="1"/>
-<wire x1="56.7796" y1="32.54513125" x2="58.086" y2="33.85153125" width="0.3048" layer="1"/>
+<wire x1="58.086" y1="34.544" x2="58.01646875" y2="34.544" width="0.3048" layer="1"/>
+<wire x1="58.01646875" y1="34.544" x2="55.88" y2="32.40753125" width="0.3048" layer="1"/>
 <wire x1="54.8990375" y1="30.48" x2="55.64351875" y2="31.22448125" width="0.3048" layer="1"/>
 <wire x1="55.64351875" y1="31.22448125" x2="55.77051875" y2="31.35148125" width="0.3048" layer="1"/>
 <wire x1="55.77051875" y1="31.35148125" x2="55.88" y2="31.4609625" width="0.3048" layer="1"/>
-<wire x1="55.88" y1="31.4609625" x2="56.7796" y2="32.3605625" width="0.3048" layer="1"/>
-<wire x1="56.7796" y1="32.3605625" x2="56.7796" y2="32.54513125" width="0.3048" layer="1"/>
+<wire x1="55.88" y1="31.4609625" x2="55.88" y2="32.40753125" width="0.3048" layer="1"/>
 <wire x1="52.8636" y1="30.48" x2="54.8990375" y2="30.48" width="0.3048" layer="1"/>
 <wire x1="45.3073" y1="29.464" x2="46.2342" y2="28.5371" width="0.3048" layer="1"/>
@@
 <mfgpreviewcolor name="substratecolor" color="0xFF786E46"/>
 </mfgpreviewcolors>
-<errors>
-</errors>
 </board>
 </drawing>

Commit message: update schematic
Parts:
- VR5: value 100K -> 50K
Changed lines of the file:
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@@
 <attribute name="VALUE" x="28.956" y="1.524" size="1.27" layer="27" font="vector" rot="R90"/>
 </element>
-<element name="VR5" library="Passive_Robotech" package="VR2C" value="100K" x="58.086" y="32.004" smashed="yes" rot="R90">
+<element name="VR5" library="Passive_Robotech" package="VR2C" value="50K" x="58.086" y="32.004" smashed="yes" rot="R90">
 <attribute name="NAME" x="56.816" y="30.734" size="1.27" layer="25" rot="R90"/>
 <attribute name="VALUE" x="63.674" y="32.512" size="1.27" layer="27" rot="R90"/>
