File: nutrino.sch (EAGLE design)
At the start: 94 parts, among them CN1 STEREO-3.5-MJ8435, CON1 MINI-USB-, IC1 TLV61046A, IC2 TAR5SB33, IC3 PCM2704, IC4 NJM4580EMP8, Q1 12M, SW1 TOGGLESW_SLIMPANEL, SW2 TOGGLESW_SLIMPANEL

Commit message: placed parts
Parts:
- added HOLE1, HOLE2, HOLE3, HOLE4: HOLE_3.2, Document_Robotech:HOLE_3.2
- R33, R34: value 10k -> 100k
- SW1, SW2: value TOGGLESW_SLIMPANEL -> SLIDESW_SS12D01G4; device Passive_Robotech:TOGGLESW_SLIMPANEL -> Passive_Robotech:SLIDESW_SS12D01G4
- U1: device rezzonics:NUTUBE_6P1 -> rezzonics:NUTUBE_6P1_1
- renumbered 100K to R34, 100K1 to R33
Connections:
- removed net POWER-GND: C10.2, C8.2, C9.2, IC2.GND
- net GND: now also C10.2, C8.2, C9.2, IC2.GND

Commit message: Board diagram completed
Connections:
- removed net +26V: C4.1, C5.1, C6.1, C7.1
- net AVCC: now also C4.1, C5.1, C6.1, C7.1
- net GND: now also CON1.SHELL
- net N$20: now also VR1.2, VR1.BR; no longer VR1.1
- net N$26: now also VR2.1, VR2.BR; no longer VR2.2
- net TUBE_L: now also VR1.1; no longer VR1.2
- net TUBE_R: now also VR2.2; no longer VR2.1
Other:
- moved on the sheet: VR1, VR2

Commit message: add image
Parts:
- VR5: value (none) -> 100K
Changed lines of the file:
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@@
 <part name="SUPPLY27" library="Supply_Robotech" deviceset="GND" device=""/>
 <part name="R34" library="Passive_Robotech" deviceset="R" device="-2012" value="100k"/>
-<part name="VR5" library="Passive_Robotech" deviceset="VR2C" device=""/>
+<part name="VR5" library="Passive_Robotech" deviceset="VR2C" device="" value="100K"/>
 <part name="C36" library="Passive_Robotech" deviceset="C" device="-2012" value="10p"/>
 <part name="R26" library="Passive_Robotech" deviceset="R" device="-4532" value="10"/>

Commit message: update schematic
Parts:
- VR5: value 100K -> 50K
Changed lines of the file:
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@@
 <part name="SUPPLY27" library="Supply_Robotech" deviceset="GND" device=""/>
 <part name="R34" library="Passive_Robotech" deviceset="R" device="-2012" value="100k"/>
-<part name="VR5" library="Passive_Robotech" deviceset="VR2C" device="" value="100K"/>
+<part name="VR5" library="Passive_Robotech" deviceset="VR2C" device="" value="50K"/>
 <part name="C36" library="Passive_Robotech" deviceset="C" device="-2012" value="10p"/>
 <part name="R26" library="Passive_Robotech" deviceset="R" device="-4532" value="10"/>
@@
 <attribute name="VALUE" x="86.995" y="22.225" size="1.778" layer="96"/>
 </instance>
-<instance part="SUPPLY2" gate="GND" x="45.72" y="50.8" smashed="yes">
-<attribute name="VALUE" x="46.355" y="50.165" size="1.778" layer="96"/>
+<instance part="SUPPLY2" gate="GND" x="43.18" y="50.8" smashed="yes">
+<attribute name="VALUE" x="43.815" y="50.165" size="1.778" layer="96"/>
 </instance>
 <instance part="C1" gate="G$1" x="30.48" y="63.5" smashed="yes">
@@
 <instance part="IC4" gate="G$2" x="365.76" y="154.94" smashed="yes" rot="MR180">
 <attribute name="NAME" x="368.3" y="151.765" size="1.778" layer="95" rot="MR180"/>
-<attribute name="VALUE" x="368.3" y="160.02" size="1.778" layer="96" rot="MR180"/>
+<attribute name="VALUE" x="363.22" y="160.02" size="1.778" layer="96" rot="MR180"/>
 </instance>
 <instance part="IC4" gate="G$3" x="365.76" y="96.52" smashed="yes" rot="MR180">
 <attribute name="NAME" x="368.3" y="93.345" size="1.778" layer="95" rot="MR180"/>
-<attribute name="VALUE" x="368.3" y="101.6" size="1.778" layer="96" rot="MR180"/>
+<attribute name="VALUE" x="363.22" y="101.6" size="1.778" layer="96" rot="MR180"/>
 </instance>
 <instance part="IC4" gate="G$1" x="345.44" y="43.18" smashed="yes">
@@
 <instance part="VR5" gate="G$1" x="360.68" y="172.72" smashed="yes">
 <attribute name="NAME" x="356.87" y="174.2186" size="1.778" layer="95"/>
-<attribute name="VALUE" x="356.87" y="161.798" size="1.778" layer="96"/>
+<attribute name="VALUE" x="356.87" y="177.038" size="1.778" layer="96"/>
 </instance>
 <instance part="VR5" gate="G$2" x="360.68" y="114.3" smashed="yes">
 <attribute name="NAME" x="356.87" y="115.7986" size="1.778" layer="95"/>
-<attribute name="VALUE" x="356.87" y="103.378" size="1.778" layer="96"/>
+<attribute name="VALUE" x="356.87" y="118.618" size="1.778" layer="96"/>
 </instance>
 <instance part="C36" gate="G$1" x="365.76" y="167.64" smashed="yes" rot="R90">
@@
 </instance>
 <instance part="R26" gate="G$1" x="381" y="154.94" smashed="yes">
-<attribute name="NAME" x="377.19" y="156.4386" size="1.778" layer="95"/>
-<attribute name="VALUE" x="377.19" y="151.638" size="1.778" layer="96"/>
+<attribute name="NAME" x="379.73" y="156.4386" size="1.778" layer="95"/>
+<attribute name="VALUE" x="379.73" y="151.638" size="1.778" layer="96"/>
 </instance>
 <instance part="C37" gate="G$1" x="388.62" y="154.94" smashed="yes" rot="R90">
 <attribute name="NAME" x="392.684" y="159.385" size="1.778" layer="95" rot="R180"/>
-<attribute name="VALUE" x="395.224" y="151.511" size="1.778" layer="96" rot="R180"/>
+<attribute name="VALUE" x="392.684" y="151.511" size="1.778" layer="96" rot="R180"/>
 </instance>
 <instance part="R27" gate="G$1" x="398.78" y="149.86" smashed="yes" rot="R90">
@@
 </instance>
 <instance part="R31" gate="G$1" x="381" y="96.52" smashed="yes">
-<attribute name="NAME" x="377.19" y="98.0186" size="1.778" layer="95"/>
-<attribute name="VALUE" x="377.19" y="93.218" size="1.778" layer="96"/>
+<attribute name="NAME" x="379.73" y="98.0186" size="1.778" layer="95"/>
+<attribute name="VALUE" x="379.73" y="93.218" size="1.778" layer="96"/>
 </instance>
 <instance part="C41" gate="G$1" x="388.62" y="96.52" smashed="yes" rot="R90">
 <attribute name="NAME" x="392.684" y="100.965" size="1.778" layer="95" rot="R180"/>
-<attribute name="VALUE" x="395.224" y="93.091" size="1.778" layer="96" rot="R180"/>
+<attribute name="VALUE" x="392.684" y="93.091" size="1.778" layer="96" rot="R180"/>
 </instance>
 <instance part="R32" gate="G$1" x="398.78" y="91.44" smashed="yes" rot="R90">
@@
 <pinref part="IC1" gate="G$1" pin="GND"/>
 <pinref part="SUPPLY2" gate="GND" pin="GND"/>
-</segment>
-<segment>
+<wire x1="43.18" y1="53.34" x2="45.72" y2="53.34" width="0.1524" layer="91"/>
+</segment>
+<segment>
